File: other/KiCad/OverlordDimmer/OverlordDimmer.kicad_pcb (KiCad board)
At the start: 2 copper layers, 155.1 x 86.1 mm, 184 parts, among them J1 Connector_Screw_Terminal_01x09, J2 USB_cable, J3 RJ45x2, J4 Connector_Screw_Terminal_01x09, J5 USB_B, J6 Conn_01x12_Female, Q1 IRF740, Q10 IRF740, Q11 IRF740, Q12 IRF740, Q13 2N3906, Q14 IRF740, Q15 2N3904, Q16 IRF740, Q17 2N3906, Q18 2N3904, Q19 IRF740, Q2 2N3904, Q20 IRF740, Q21 2N7002E, Q22 2N7002E, Q23 2N3904, Q24 IRF740, Q25 IRF740, Q26 2N3904, Q27 IRF740, Q28 IRF740, Q29 2N3906, Q3 2N3906, Q30 2N3904, Q31 2N3906, Q32 IRF740, Q33 2N3906, Q34 2N3904, Q35 IRF740, Q36 IRF740, Q37 2N3904, Q38 2N3906, Q39 IRF740, Q4 IRF740, Q40 IRF740, Q41 2N3906, Q42 IRF740, Q43 NPN, Q44 BC817, Q45 NPN, Q5 IRF740, Q6 2N3906, Q7 2N3904, Q8 2N3904, Q9 2N3906, U1 4N25, U10 4N25, U11 4N25, U12 4N35, U2 4N25, U3 4N25, U4 SN65HVD230, U5 4N25, U6 4N25, U7 4N25, U8 4N25, U9 4N25

Commit message: Finalised ver1.0 revA of PCB
Parts:
- added D18: SBR1A40S1, Diode_SMD:D_SOD-123, F.Cu at (100.6, 94.1)
- Q43, Q45: value NPN -> 2SC4061KT146N
- R12, R13: footprint Resistor_SMD:R_1812_4532Metric_Pad1.30x3.40mm_HandSolder -> Resistor_SMD:R_0402_1005Metric_Pad0.72x0.64mm_HandSolder
- R15, R27: footprint Resistor_SMD:R_0805_2012Metric_Pad1.20x1.40mm_HandSolder -> Resistor_SMD:R_0402_1005Metric_Pad0.72x0.64mm_HandSolder
- R56: footprint Resistor_SMD:R_1210_3225Metric_Pad1.30x2.65mm_HandSolder -> Resistor_SMD:R_0805_2012Metric_Pad1.20x1.40mm_HandSolder
- R60: footprint Resistor_SMD:R_0805_2012Metric_Pad1.20x1.40mm_HandSolder -> Resistor_SMD:R_1210_3225Metric_Pad1.30x2.65mm_HandSolder
- R61: footprint Resistor_SMD:R_0402_1005Metric_Pad0.72x0.64mm_HandSolder -> Resistor_SMD:R_1210_3225Metric_Pad1.30x2.65mm_HandSolder
- R64, R65, R66: footprint Resistor_SMD:R_0805_2012Metric_Pad1.20x1.40mm_HandSolder -> Resistor_SMD:R_1206_3216Metric_Pad1.30x1.75mm_HandSolder
- moved R45 5.01 mm to (130.1, 30.8)
- moved R60 3.07 mm to (156.5, 47.0)
- moved R15 2.91 mm to (57.0, 104.9)
- moved R12 2.30 mm to (72.5, 86.7), turned to 180 degrees
- moved DbgGND1 2.29 mm to (101.1, 98.5)
- moved DbgURX1 2.29 mm to (101.1, 106.1)
- moved DbgUTX1 2.29 mm to (101.1, 102.3)
- moved R61 2.07 mm to (156.6, 52.5)
- moved R27 1.70 mm to (64.7, 106.2)
Connections:
- J2 pad 4: Net-(J2-Pin_4) -> Net-(D18-K)
- J5 pad 1: Net-(J2-Pin_4) -> Net-(D18-A)
Routing:
- net L: track 399.2 -> 369.4 mm
- net Net-(D18-A): track 0.00 -> 10.0 mm
- net Net-(D18-K): track 0.00 -> 7.80 mm
- net UART_TX_0: track 167.0 -> 161.1 mm, vias 0 -> 1
- net Net-(J2-Pin_4): track 5.10 -> 0.00 mm
- net Net-(Q43-B): track 7.82 -> 12.7 mm
- net +5V: track 130.0 -> 126.5 mm
- net +12V: track 21.7 -> 18.3 mm
- net CAN_TX: track 187.0 -> 184.3 mm, vias 1 -> 2
- net Net-(D15-A): track 16.5 -> 18.6 mm
- net Net-(D14-K): track 10.0 -> 11.9 mm
- net VCC: track 185.5 -> 187.2 mm
- net Net-(11-Pin_2): track 5.67 -> 7.30 mm
- net CAN_H: track 59.8 -> 61.5 mm
- net TRGR1: track 184.8 -> 186.4 mm
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